File: oled-controller.kicad_pcb (KiCad board)
At the start: 2 copper layers, 43.2 x 41.9 mm, 11 parts, among them J1 Wuerth FFC socket (slave), J2 PMOD Master, J3 adafruit-1.5inch-Color-OLED-B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, J4 10-Pin ARM Debug, J5 USB_B_Mini, U1 STM32F446RETx

Commit message: Added two LEDs
Parts:
- added C4: 100nF, Capacitor_SMD:C_0603_1608Metric_Pad1.05x0.95mm_HandSolder, B.Cu at (168.0, 67.7)
- added D1: LED, Diode_SMD:D_0603_1608Metric_Pad1.05x0.95mm_HandSolder, B.Cu at (182.9, 96.5)
- added D2: LED, Diode_SMD:D_0603_1608Metric_Pad1.05x0.95mm_HandSolder, B.Cu at (152.4, 96.5)
- added R3: R_Small, Resistor_SMD:R_0603_1608Metric_Pad1.05x0.95mm_HandSolder, B.Cu at (179.1, 96.5)
- added R4: R_Small, Resistor_SMD:R_0603_1608Metric_Pad1.05x0.95mm_HandSolder, B.Cu at (156.6, 96.5)
- J1: value Wuerth FFC socket (slave) -> Wuerth FFC socket (slave configuration)
- moved J5 0.38 mm to (183.3, 82.5)
Connections:
- U1 pad 33: Net-(U1-Pad33) -> /Blinky
Routing:
- net +3V3: track 76.4 -> 96.9 mm
- net /Blinky: track 0.00 -> 11.9 mm, vias 0 -> 1
- net GND: track 25.8 -> 34.6 mm
- net Net-(D2-Pad2): track 0.00 -> 2.45 mm

Commit message: PCB: Final adjustments
Routing:
- net +3V3: track 96.9 -> 122.7 mm, vias 2 -> 3
- net GND: track 34.6 -> 34.9 mm, vias 44 -> 50
- net (no net): vias 3 -> 0
- removed copper zone on B.Cu, net Net-(J5-Pad6)
Other:
- rule trace_min: 0.2 -> 0.16
